File: RPi Hat RF Transmitter V1.sch (KiCad schematic (older format))
At the start: 67 parts, among them CON1 Sig_In, CON2 SMA-, CON3 Sig_In, CON4 Sig_In, CON5 SMA-, IC1 HMC241AQS16E, IC2 HMC241AQS16E, IC3 SN74HC139PW, J1 Conn_01x04_Male, J2 Conn_01x04_Male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

Commit message: removes digital switch and puts mechanical switch
Parts:
- removed C19: 0.1uF, Capacitor_SMD:C_0805_2012Metric_Pad1.15x1.40mm_HandSolder, symbol Device:C
- removed D1: Blue, LED_SMD:LED_0805_2012Metric_Pad1.15x1.40mm_HandSolder, symbol Device:LED
- removed D2: Green, LED_SMD:LED_0805_2012Metric_Pad1.15x1.40mm_HandSolder, symbol Device:LED
- removed D3: Orange, LED_SMD:LED_0805_2012Metric_Pad1.15x1.40mm_HandSolder, symbol Device:LED
- removed D4: Yellow, LED_SMD:LED_0805_2012Metric_Pad1.15x1.40mm_HandSolder, symbol Device:LED
- removed D7: Red, LED_SMD:LED_0805_2012Metric_Pad1.15x1.40mm_HandSolder, symbol Device:LED
- removed IC1, IC2: HMC241AQS16E, SamacSys_Parts:SOP64P600X175-16N, symbol SamacSys_Parts:HMC241AQS16E
- removed IC3: SN74HC139PW, Package_SO:SOIC-16_3.9x9.9mm_P1.27mm, symbol SamacSys_Parts:SN74HC139PW
- removed J1: Conn_01x04_Male, Connector_PinHeader_2.54mm:PinHeader_1x04_P2.54mm_Vertical, symbol Connector:Conn_01x04_Male
- removed J5, J7: Conn_01x03_Male, Connector_PinHeader_2.54mm:PinHeader_1x03_P2.54mm_Vertical, symbol Connector:Conn_01x03_Male
- removed JP2, JP3: Jumper, Connector_PinHeader_2.54mm:PinHeader_1x02_P2.54mm_Vertical, symbol Device:Jumper
- removed R11, R12, R13, R14, R15: 330, Resistor_SMD:R_0805_2012Metric_Pad1.15x1.40mm_HandSolder, symbol Device:R
- removed U2: 74AUC2G04, Package_TO_SOT_SMD:SOT-23-6_Handsoldering, symbol 74xGxx:74AUC2G04
- added SW1, SW2: SW_Coded, VK_Cus_KiCad:1x4_switch, symbol Switch:SW_Coded
Connections:
- net RF1_IN: now also SW1.2 (D0)
- net RF1_OUT: now also SW2.5 (D3)
- net RF2_IN: now also SW1.3 (D1)
- net RF2_OUT: now also SW2.4 (D2)
- net RF3_IN: now also SW1.4 (D2)
- net RF3_OUT: now also SW2.3 (D1)
- net RF4_IN: now also SW1.5 (D3)
- net RF4_OUT: now also SW2.2 (D0)
- net RF_ANT_OUT: now also SW1.1 (CM)
- net GPIO17: no longer names the net of J3.11 (BCM17)
- net GPIO22: no longer names the net of J3.15 (BCM22)
- net GPIO27: no longer names the net of J3.13 (BCM27)
- net GPIO4 renamed RF_IN_SWITCH
- net RF_IN_SWITCH: now also SW2.1 (CM)
- no-connect marks 36 -> 32

Commit message: goes on proto production here
Parts:
- added FL4: LFCN-180, Filter:Filter_Mini-Circuits_FV1206, symbol RF_Filter:LFCN-180
- added JP2, JP3: Jumper, Connector_PinHeader_2.54mm:PinHeader_1x02_P2.54mm_Vertical, symbol Device:Jumper
Connections:
- net GND: now also FL4.2 (GND), FL4.4 (GND)
- net RF4_IN: now also FL4.3 (OUT)
- net RF4_OUT: now also FL4.1 (IN)
- net RF_ANT_OUT: now also JP3.2; no longer SW1.1 (CM)
- net RF_IN_SWITCH: now also JP2.1; no longer J3.7 (BCM4)
- new net: JP3.1, SW1.1 (CM)
- new net RF_RPI: J3.7 (BCM4), JP2.2
Other:
- moved on the sheet: CON4
Changed lines of the file:
@@
 Text GLabel 1275 9850 0    50   Input Italic 0
 RF4_OUT
-Text GLabel 4000 9850 2    50   Input Italic 0
+Text GLabel 3300 9850 2    50   Input Italic 0
 RF4_IN
 Wire Notes Line
@@
 L vk_custom_kicad:SMA- CON4
 U 1 1 5DD39EB4
-P 3350 9850
-F 0 "CON4" V 3390 9880 50  0000 L CNN
-F 1 "Sig_In" V 3299 9880 50  0000 L CNN
-F 2 "Connector_Coaxial:SMA_Amphenol_132291-12_Vertical" V 3350 9650 50  0001 C CNN
-F 3 "JOHNSON COMPONENTS" H 3500 9700 50  0001 L BNN
-F 4 "91B6105" H 3750 9600 50  0001 L BNN "Field4"
-F 5 "1339835" H 3750 9600 50  0001 L BNN "Field5"
-F 6 "142-0701-871" H 3500 9700 50  0001 L BNN "Field6"
-	1    3350 9850
+P 2650 9850
+F 0 "CON4" V 2690 9880 50  0000 L CNN
+F 1 "Sig_In" V 2599 9880 50  0000 L CNN
+F 2 "Connector_Coaxial:SMA_Amphenol_132291-12_Vertical" V 2650 9650 50  0001 C CNN
+F 3 "JOHNSON COMPONENTS" H 2800 9700 50  0001 L BNN
+F 4 "91B6105" H 3050 9600 50  0001 L BNN "Field4"
+F 5 "1339835" H 3050 9600 50  0001 L BNN "Field5"
+F 6 "142-0701-871" H 2800 9700 50  0001 L BNN "Field6"
+	1    2650 9850
 	0    -1   -1   0
 $EndComp
@@
 L power:GND #PWR06
 U 1 1 5DD39EBA
-P 3700 10025
-F 0 "#PWR06" H 3700 9775 50  0001 C CNN
-F 1 "GND" H 3705 9852 50  0000 C CNN
-F 2 "" H 3700 10025 50  0001 C CNN
-F 3 "" H 3700 10025 50  0001 C CNN
-	1    3700 10025
+P 3000 10025
+F 0 "#PWR06" H 3000 9775 50  0001 C CNN
+F 1 "GND" H 3005 9852 50  0000 C CNN
+F 2 "" H 3000 10025 50  0001 C CNN
+F 3 "" H 3000 10025 50  0001 C CNN
+	1    3000 10025
 	-1   0    0    -1
 $EndComp
 Wire Wire Line
-	3650 9950 3700 9950
-Wire Wire Line
-	3700 9950 3700 10025
+	2950 9950 3000 9950
+Wire Wire Line
+	3000 9950 3000 10025
 $Comp
 L Device:R R10
@@
 	1275 9850 1575 9850
 Wire Wire Line
-	3650 9850 4000 9850
+	2950 9850 3300 9850
 Wire Wire Line
 	7650 3075 8000 3075
@@
 Text GLabel 12625 2975 0    50   Input Italic 0
 RF4_OUT
-Text GLabel 12625 3125 0    50   Input ~ 0
+Text GLabel 11925 3475 0    50   Input ~ 0
 RF_IN_SWITCH
-Text GLabel 14775 2675 2    50   Input ~ 0
+Text GLabel 15375 2675 2    50   Input ~ 0
 RF_ANT_OUT
 Text GLabel 14775 2825 2    50   Input Italic 0
@@
 Text GLabel 14775 3125 2    50   Input Italic 0
 RF4_IN
-Text GLabel 1200 1875 0    50   Input ~ 0
-RF_IN_SWITCH
 NoConn ~ 2100 2075
 NoConn ~ 2100 2175
 NoConn ~ 2100 2275
+$Comp
+L RF_Filter:LFCN-180 FL4
+U 1 1 5DA66447
+P 4800 9850
+F 0 "FL4" H 4800 10317 50  0000 C CNN
+F 1 "LFCN-180" H 4800 10226 50  0000 C CNN
+F 2 "Filter:Filter_Mini-Circuits_FV1206" H 4800 10350 50  0001 C CNN
+F 3 "https://www.minicircuits.com/pdfs/LFCN-180+.pdf" H 4800 9850 50  0001 C CNN
+	1    4800 9850
+	1    0    0    -1
+$EndComp
+Text GLabel 5200 9850 2    50   Input Italic 0
+RF4_IN
+Text GLabel 4400 9850 0    50   Input Italic 0
+RF4_OUT
+$Comp
+L power:GND #PWR0101
+U 1 1 5DA8745E
+P 4800 10250
+F 0 "#PWR0101" H 4800 10000 50  0001 C CNN
+F 1 "GND" H 4805 10077 50  0000 C CNN
+F 2 "" H 4800 10250 50  0001 C CNN
+F 3 "" H 4800 10250 50  0001 C CNN
+	1    4800 10250
+	-1   0    0    -1
+$EndComp
+$Comp
+L Device:Jumper JP2
+U 1 1 5DA89EAB
+P 12225 3125
+F 0 "JP2" H 12225 3389 50  0000 C CNN
+F 1 "Jumper" H 12225 3298 50  0000 C CNN
+F 2 "Connector_PinHeader_2.54mm:PinHeader_1x02_P2.54mm_Vertical" H 12225 3125 50  0001 C CNN
+F 3 "~" H 12225 3125 50  0001 C CNN
+	1    12225 3125
+	-1   0    0    1
+$EndComp
+$Comp
+L Device:Jumper JP3
+U 1 1 5DAA0E83
+P 15075 2675
+F 0 "JP3" H 15075 2939 50  0000 C CNN
+F 1 "Jumper" H 15075 2848 50  0000 C CNN
+F 2 "Connector_PinHeader_2.54mm:PinHeader_1x02_P2.54mm_Vertical" H 15075 2675 50  0001 C CNN
+F 3 "~" H 15075 2675 50  0001 C CNN
+	1    15075 2675
+	1    0    0    -1
+$EndComp
+Wire Wire Line
+	12525 3125 12550 3125
+Text GLabel 11925 3125 0    50   Input ~ 0
+RF_RPI
+Text GLabel 1200 1875 0    50   Input ~ 0
+RF_RPI
+Wire Wire Line
+	11925 3475 12550 3475
+Wire Wire Line
+	12550 3475 12550 3125
+Connection ~ 12550 3125
+Wire Wire Line
+	12550 3125 12625 3125
 $EndSCHEMATC
